File: Kicad/TohokuMouse2016.sch (KiCad schematic (older format))
At the start: 77 parts, among them P1 BATTERY_CON, P2 DOWNLOAD, P3 L_MOTOR, P4 R_MOTOR, P5 L_ENC_MAIN, P6 R_ENC_MAIN, P7 L_ENC_SUB, P8 R_ENC_SUB, Q1 LTR-4206E, Q2 RUM003N02, Q3 LTR-4206E, Q4 RUM003N02, Q5 LTR-4206E, Q6 LTR-4206E, Q7 RUM003N02, Q8 ZXM62P02E6, Q9 RUM003N02, SW1 MAIN_SW, SW2 PUSH_SW, U1 MPU-6500, U2 AP7333-28SRG-7, U3 AP7333-28SRG-7, U4 R5F5631MCDFL, U5 DRV8836, U6 AS5055, U7 AS5055, X1 CSTCE12M0G55-R0

Commit message: Ready to PCB edit.
Parts:
- C1, C10, C11, C12, C13, C6, C7, C9, D4, D6, D7, D8: footprint ~ -> MicroMouse:Chip_2012
- C2, C3, C4, C5, C8, R1, R10, R11, R12, R13, R14, R15, R16, R17, R18, R19, R2, R20, R21, R22, R23, R24, R25, R26, R27, R3, R4, R5, R6, R7, R8, R9: footprint ~ -> MicroMouse:Chip_1005
- D1, D2, D3, D5: footprint ~ -> MicroMouse:TSAL4400
- L1, L2: footprint ~ -> MicroMouse:VLCF4018_2
- P1: footprint (none) -> MicroMouse:BATT_CON
- P2: footprint (none) -> MicroMouse:Download
- P3, P4: footprint (none) -> MicroMouse:MotorConnect
- P5, P6: footprint (none) -> MicroMouse:Pad6_8mm_MAIN
- P7, P8: footprint (none) -> MicroMouse:Pad6_8mm_SUB
- Q1, Q3, Q5, Q6: footprint ~ -> MicroMouse:LTR_4206E; symbol OPTO_NPN -> OPTO_NPN-RESCUE-TohokuMouse2016
- Q2, Q4, Q7, Q9: footprint ~ -> MicroMouse:RUM003N02
- Q8: footprint ~ -> MicroMouse:ZXM62P02E6
- SW1: footprint ~ -> MicroMouse:SW_SPDT_PCM12
- SW2: footprint ~ -> MicroMouse:SW_SPST_EVQPE1
- U1: footprint MODULE -> MicroMouse:MPU6500
- U2, U3: footprint ~ -> MicroMouse:AP7333_xxSRG
- U4: footprint MODULE -> MicroMouse:R5F5631MCDFL
- U5: footprint MODULE -> MicroMouse:DRV8836
- U6, U7: footprint MODULE -> MicroMouse:AS5055
- X1: footprint (none) -> MicroMouse:CSTE12M0G55_R0
Connections:
- net VEE: now also Q1.2 (C), Q3.2 (C), Q5.2 (C), Q6.2 (C); no longer Q1.3 (C), Q3.3 (C), Q5.3 (C), Q6.3 (C)

Commit message: Added mech data.
Parts:
- P5, P6: footprint MicroMouse:Pad6_8mm_MAIN -> MicroMouse:EncConn
- P7, P8: footprint MicroMouse:Pad6_8mm_SUB -> MicroMouse:EncConn
Connections:
- net batt_con: now reaches P1.2, Q8.3 (S), SW1.1
Changed lines of the file:
@@
 F 0 "P7" V 10600 1950 60  0000 C CNN
 F 1 "L_ENC_SUB" V 10700 1950 60  0000 C CNN
-F 2 "MicroMouse:Pad6_8mm_SUB" H 10650 1950 60  0001 C CNN
+F 2 "MicroMouse:EncConn" H 10650 1950 60  0001 C CNN
 F 3 "" H 10650 1950 60  0000 C CNN
 	1    10650 1950
@@
 F 0 "P8" V 10600 4300 60  0000 C CNN
 F 1 "R_ENC_SUB" V 10700 4300 60  0000 C CNN
-F 2 "MicroMouse:Pad6_8mm_SUB" H 10650 4300 60  0001 C CNN
+F 2 "MicroMouse:EncConn" H 10650 4300 60  0001 C CNN
 F 3 "" H 10650 4300 60  0000 C CNN
 	1    10650 4300
@@
 F 0 "P5" V 10250 1950 60  0000 C CNN
 F 1 "L_ENC_MAIN" V 10350 1950 60  0000 C CNN
-F 2 "MicroMouse:Pad6_8mm_MAIN" H 10300 1950 60  0001 C CNN
+F 2 "MicroMouse:EncConn" H 10300 1950 60  0001 C CNN
 F 3 "" H 10300 1950 60  0000 C CNN
 	1    10300 1950
@@
 F 0 "P6" V 10250 4300 60  0000 C CNN
 F 1 "R_ENC_MAIN" V 10350 4300 60  0000 C CNN
-F 2 "MicroMouse:Pad6_8mm_MAIN" H 10300 4300 60  0001 C CNN
+F 2 "MicroMouse:EncConn" H 10300 4300 60  0001 C CNN
 F 3 "" H 10300 4300 60  0000 C CNN
 	1    10300 4300
@@
 	11350 1450 11350 1800
 Connection ~ 11350 1800
+Text Label 1850 900  0    60   ~ 0
+batt_con
 $EndSCHEMATC

Commit message: update mech data.
Parts:
- U2, U3: footprint MicroMouse:AP7333_xxSRG -> MicroMouse:AP7333_xxSR
Changed lines of the file:
@@
 F 0 "U2" H 4950 754 60  0000 C CNN
 F 1 "AP7333-28SRG-7" H 4800 1150 60  0000 C CNN
-F 2 "MicroMouse:AP7333_xxSRG" H 4800 950 60  0001 C CNN
+F 2 "MicroMouse:AP7333_xxSR" H 4800 950 60  0001 C CNN
 F 3 "~" H 4800 950 60  0000 C CNN
 	1    4800 950
@@
 F 0 "U3" H 4950 1754 60  0000 C CNN
 F 1 "AP7333-28SRG-7" H 4800 2150 60  0000 C CNN
-F 2 "MicroMouse:AP7333_xxSRG" H 4800 1950 60  0001 C CNN
+F 2 "MicroMouse:AP7333_xxSR" H 4800 1950 60  0001 C CNN
 F 3 "~" H 4800 1950 60  0000 C CNN
 	1    4800 1950

Commit message: Update circuitdiagram.
Connections:
- net FR_ON: now also U4.22 (PC6); no longer U4.13 (P17)
- net GND: now also R23.1, R25.1, R27.1
- net LED0: now also D6.1 (A); no longer D6.2 (K)
- net LED1: now also D7.1 (A); no longer D7.2 (K)
- net LED2: now also D8.1 (A); no longer D8.2 (K)
- net LS_ON: now also U4.13 (P17); no longer U4.22 (PC6)
- net VCC: no longer R23.1, R25.1, R27.1
- net at R23.2: now also D6.2 (K); no longer D6.1 (A)
- net at R25.2: now also D7.2 (K); no longer D7.1 (A)
- net at R27.2: now also D8.2 (K); no longer D8.1 (A)
Changed lines of the file:
@@
 FL_ON
 Text Label 7500 4850 0    60   ~ 0
-FR_ON
+LS_ON
 Entry Wire Line
 	7950 3950 8050 4050
@@
 	7950 3850 8050 3950
 Text Label 7500 3950 0    60   ~ 0
-LS_ON
+FR_ON
 Text Label 7500 3850 0    60   ~ 0
 RS_ON
@@
 F 3 "~" H 6700 9800 60  0000 C CNN
 	1    6700 9800
-	0    1    1    0
+	0    -1   -1   0
 $EndComp
 $Comp
@@
 	1    0    0    -1
 $EndComp
-$Comp
-L VCC #PWR049
-U 1 1 56829635
-P 6700 8700
-F 0 "#PWR049" H 6700 8800 30  0001 C CNN
-F 1 "VCC" H 6700 8800 30  0000 C CNN
-F 2 "" H 6700 8700 60  0000 C CNN
-F 3 "" H 6700 8700 60  0000 C CNN
-	1    6700 8700
-	1    0    0    -1
-$EndComp
 Entry Wire Line
 	6400 8200 6500 8300
@@
 F 3 "~" H 7300 9800 60  0000 C CNN
 	1    7300 9800
-	0    1    1    0
+	0    -1   -1   0
 $EndComp
 $Comp
@@
 	1    0    0    -1
 $EndComp
-$Comp
-L VCC #PWR050
-U 1 1 56829A91
-P 7300 8700
-F 0 "#PWR050" H 7300 8800 30  0001 C CNN
-F 1 "VCC" H 7300 8800 30  0000 C CNN
-F 2 "" H 7300 8700 60  0000 C CNN
-F 3 "" H 7300 8700 60  0000 C CNN
-	1    7300 8700
-	1    0    0    -1
-$EndComp
 Entry Wire Line
 	7000 8200 7100 8300
@@
 F 3 "~" H 7900 9800 60  0000 C CNN
 	1    7900 9800
-	0    1    1    0
+	0    -1   -1   0
 $EndComp
 $Comp
@@
 F 3 "~" H 7900 9150 30  0000 C CNN
 	1    7900 9150
-	1    0    0    -1
-$EndComp
-$Comp
-L VCC #PWR051
-U 1 1 5682A2C5
-P 7900 8700
-F 0 "#PWR051" H 7900 8800 30  0001 C CNN
-F 1 "VCC" H 7900 8800 30  0000 C CNN
-F 2 "" H 7900 8700 60  0000 C CNN
-F 3 "" H 7900 8700 60  0000 C CNN
-	1    7900 8700
 	1    0    0    -1
 $EndComp
@@
 Text Label 1850 900  0    60   ~ 0
 batt_con
+$Comp
+L GND-RESCUE-TohokuMouse2016 #PWR?
+U 1 1 578774F9
+P 6850 8750
+F 0 "#PWR?" H 6850 8750 30  0001 C CNN
+F 1 "GND" H 6850 8680 30  0001 C CNN
+F 2 "" H 6850 8750 60  0000 C CNN
+F 3 "" H 6850 8750 60  0000 C CNN
+	1    6850 8750
+	1    0    0    -1
+$EndComp
+$Comp
+L GND-RESCUE-TohokuMouse2016 #PWR?
+U 1 1 5787771F
+P 7450 8750
+F 0 "#PWR?" H 7450 8750 30  0001 C CNN
+F 1 "GND" H 7450 8680 30  0001 C CNN
+F 2 "" H 7450 8750 60  0000 C CNN
+F 3 "" H 7450 8750 60  0000 C CNN
+	1    7450 8750
+	1    0    0    -1
+$EndComp
+$Comp
+L GND-RESCUE-TohokuMouse2016 #PWR?
+U 1 1 57877811
+P 8050 8750
+F 0 "#PWR?" H 8050 8750 30  0001 C CNN
+F 1 "GND" H 8050 8680 30  0001 C CNN
+F 2 "" H 8050 8750 60  0000 C CNN
+F 3 "" H 8050 8750 60  0000 C CNN
+	1    8050 8750
+	1    0    0    -1
+$EndComp
+Wire Wire Line
+	6700 8700 6850 8700
+Wire Wire Line
+	6850 8700 6850 8750
+Wire Wire Line
+	7300 8700 7450 8700
+Wire Wire Line
+	7450 8700 7450 8750
+Wire Wire Line
+	7900 8700 8050 8700
+Wire Wire Line
+	8050 8700 8050 8750
 $EndSCHEMATC
