File: Kicad/TohokuMouse2016.kicad_pcb (KiCad board)
At the start: 2 copper layers, 0 parts

Commit message: Ready to PCB edit.
Parts:
- added C1: 10n, MicroMouse:Chip_2012, F.Cu at (219.9, 120.5)
- added C10: 10u, MicroMouse:Chip_2012, F.Cu at (215.1, 127.9)
- added C11: 10u, MicroMouse:Chip_2012, F.Cu at (208.4, 134.3)
- added C12: 10u, MicroMouse:Chip_2012, F.Cu at (199.6, 137.6)
- added C13: 10u, MicroMouse:Chip_2012, F.Cu at (210.9, 127.9)
- added C2: 0.1u, MicroMouse:Chip_1005, F.Cu at (197.8, 149.2)
- added C3: 0.1u, MicroMouse:Chip_1005, F.Cu at (201.7, 143.6)
- added C4: 0.1u, MicroMouse:Chip_1005, F.Cu at (207.8, 140.3)
- added C5: 0.1u, MicroMouse:Chip_1005, F.Cu at (197.8, 143.6)
- added C6: 10u, MicroMouse:Chip_2012, F.Cu at (189.4, 151.9)
- added C7: 10u, MicroMouse:Chip_2012, F.Cu at (193.7, 149.1)
- added C8: 0.1u, MicroMouse:Chip_1005, F.Cu at (196.5, 124.1)
- added C9: 10u, MicroMouse:Chip_2012, F.Cu at (193.7, 142.7)
- added D1: TSAL4400, MicroMouse:TSAL4400, F.Cu at (178.2, 152.9)
- added D2: TSAL4400, MicroMouse:TSAL4400, F.Cu at (202.4, 132.9)
- added D3: TSAL4400, MicroMouse:TSAL4400, F.Cu at (178.2, 150.1)
- added D4: LED, MicroMouse:Chip_2012, F.Cu at (185.3, 151.9)
- added D5: TSAL4400, MicroMouse:TSAL4400, F.Cu at (177.9, 155.6)
- added D6: LED, MicroMouse:Chip_2012, F.Cu at (206.8, 127.9)
- added D7: LED, MicroMouse:Chip_2012, F.Cu at (203.7, 137.6)
- added D8: LED, MicroMouse:Chip_2012, F.Cu at (227.1, 117.8)
- added L1: VLCF5024T-470MR40-2, MicroMouse:VLCF4018_2, F.Cu at (164.9, 117.0)
- added L2: VLCF5024T-470MR40-2, MicroMouse:VLCF4018_2, F.Cu at (164.9, 121.9)
- added P1: BATTERY_CON, MicroMouse:BATT_CON, F.Cu at (193.4, 136.9)
- added P2: DOWNLOAD, MicroMouse:Download, F.Cu at (159.7, 155.9)
- added P3: L_MOTOR, MicroMouse:MotorConnect, F.Cu at (221.4, 115.9)
- added P4: R_MOTOR, MicroMouse:MotorConnect, F.Cu at (186.9, 147.3)
- added P5: L_ENC_MAIN, MicroMouse:Pad6_8mm_MAIN, F.Cu at (172.2, 140.8)
- added P6: R_ENC_MAIN, MicroMouse:Pad6_8mm_MAIN, F.Cu at (174.8, 133.3)
- added P7: L_ENC_SUB, MicroMouse:Pad6_8mm_SUB, F.Cu at (213.2, 117.8)
- added P8: R_ENC_SUB, MicroMouse:Pad6_8mm_SUB, F.Cu at (193.8, 131.5)
- added Q1: LTR-4206E, MicroMouse:LTR_4206E, F.Cu at (181.5, 138.4)
- added Q2: RUM003N02, MicroMouse:RUM003N02, F.Cu at (189.7, 124.9)
- added Q3: LTR-4206E, MicroMouse:LTR_4206E, F.Cu at (169.6, 151.9)
- added Q4: RUM003N02, MicroMouse:RUM003N02, F.Cu at (194.7, 117.9)
- added Q5: LTR-4206E, MicroMouse:LTR_4206E, F.Cu at (169.6, 149.1)
- added Q6: LTR-4206E, MicroMouse:LTR_4206E, F.Cu at (172.1, 145.9)
- added Q7: RUM003N02, MicroMouse:RUM003N02, F.Cu at (160.2, 151.2)
- added Q8: ZXM62P02E6, MicroMouse:ZXM62P02E6, F.Cu at (179.7, 125.5)
- added Q9: RUM003N02, MicroMouse:RUM003N02, F.Cu at (184.5, 132.9)
- added R1: 1k, MicroMouse:Chip_1005, F.Cu at (216.2, 139.5)
- added R10: 1k, MicroMouse:Chip_1005, F.Cu at (197.6, 154.8)
- added R11: 1k, MicroMouse:Chip_1005, F.Cu at (219.3, 132.1)
- added R12: 100k, MicroMouse:Chip_1005, F.Cu at (205.9, 145.9)
- added R13: 1k, MicroMouse:Chip_1005, F.Cu at (222.5, 126.5)
- added R14: 4.7, MicroMouse:Chip_1005, F.Cu at (215.8, 133.9)
- added R15: 1k, MicroMouse:Chip_1005, F.Cu at (226.6, 123.8)
- added R16: 100k, MicroMouse:Chip_1005, F.Cu at (193.7, 155.1)
- added R17: 470, MicroMouse:Chip_1005, F.Cu at (212.2, 133.9)
- added R18: 4.7, MicroMouse:Chip_1005, F.Cu at (218.9, 126.5)
- added R19: 100k, MicroMouse:Chip_1005, F.Cu at (212.6, 139.5)
- added R2: 1k, MicroMouse:Chip_1005, F.Cu at (204.2, 151.5)
- added R20: 100k, MicroMouse:Chip_1005, F.Cu at (231.3, 117.4)
- added R21: 10k, MicroMouse:Chip_1005, F.Cu at (217.7, 145.1)
- added R22: 10k, MicroMouse:Chip_1005, F.Cu at (230.4, 134.2)
- added R23: 470, MicroMouse:Chip_1005, F.Cu at (214.1, 145.1)
- added R24: 10k, MicroMouse:Chip_1005, F.Cu at (225.9, 135.0)
- added R25: 470, MicroMouse:Chip_1005, F.Cu at (207.4, 151.5)
- added R26: 10k, MicroMouse:Chip_1005, F.Cu at (219.4, 137.7)
- added R27: 470, MicroMouse:Chip_1005, F.Cu at (230.4, 128.6)
- added R3: 100k, MicroMouse:Chip_1005, F.Cu at (210.2, 145.9)
- added R4: 4.7, MicroMouse:Chip_1005, F.Cu at (222.6, 132.1)
- added R5: 1k, MicroMouse:Chip_1005, F.Cu at (200.8, 154.8)
- added R6: 1k, MicroMouse:Chip_1005, F.Cu at (223.4, 120.1)
- added R7: 100k, MicroMouse:Chip_1005, F.Cu at (231.3, 123.0)
- added R8: 4.7, MicroMouse:Chip_1005, F.Cu at (201.3, 149.2)
- added R9: 100k, MicroMouse:Chip_1005, F.Cu at (226.4, 129.4)
- added SW1: MAIN_SW, MicroMouse:SW_SPDT_PCM12, F.Cu at (204.2, 118.9)
- added SW2: PUSH_SW, MicroMouse:SW_SPST_EVQPE1, F.Cu at (187.4, 143.6)
- added U1: MPU-6500, MicroMouse:MPU6500, F.Cu at (169.5, 155.3)
- added U2: AP7333-28SRG-7, MicroMouse:AP7333_xxSRG, F.Cu at (162.7, 127.5)
- added U3: AP7333-28SRG-7, MicroMouse:AP7333_xxSRG, F.Cu at (162.7, 132.1)
- added U4: R5F5631MCDFL, MicroMouse:R5F5631MCDFL, F.Cu at (161.4, 140.7)
- added U5: DRV8836, MicroMouse:DRV8836, F.Cu at (212.4, 121.6)
- added U6: AS5055, MicroMouse:AS5055, F.Cu at (201.6, 127.1)
- added U7: AS5055, MicroMouse:AS5055, F.Cu at (180.1, 144.3)
- added X1: CSTCE12M0G55-R0, MicroMouse:CSTE12M0G55_R0, F.Cu at (182.2, 118.2)

Commit message: Added mech data.
Parts:
- P5, P6: footprint MicroMouse:Pad6_8mm_MAIN -> MicroMouse:EncConn
- P7, P8: footprint MicroMouse:Pad6_8mm_SUB -> MicroMouse:EncConn
- moved P7 95.2 mm to (120.6, 139.8)
- moved D8 94.4 mm to (135.1, 139.3)
- moved R15 89.4 mm to (139.0, 141.9)
- moved U5 82.0 mm to (131.2, 133.0)
- moved R9 80.2 mm to (147.3, 141.9)
- moved SW1 78.3 mm to (125.9, 122.3)
- moved C11 77.5 mm to (131.0, 139.3)
- moved R7 75.8 mm to (156.2, 132.5)
- moved P3 75.5 mm to (146.0, 120.0)
- moved C10 73.0 mm to (142.1, 130.3)
- moved C12 72.8 mm to (126.8, 139.3)
- moved Q9 70.8 mm to (113.9, 127.0)
- moved P8 70.4 mm to (123.4, 134.2)
- moved R19 69.7 mm to (142.9, 141.9)
- moved R17 69.3 mm to (142.9, 136.3)
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Connections:
- net Net-(P1-Pad2) renamed /batt_con
Other:
- board outline added: 67.6 x 35 mm
- net class Battery added: clearance 0.254, trace_width 2, via_dia 0.889, via_drill 0.635
- net class Bold added: clearance 0.254, trace_width 1, via_dia 0.889, via_drill 0.635
- rule via_min_drill: 0.508 -> 0.635

Commit message: update mech data.
Parts:
- U2, U3: footprint MicroMouse:AP7333_xxSRG -> MicroMouse:AP7333_xxSR
- moved R1 77.9 mm to (115.6, 70.4)
- moved D1 74.0 mm to (123.7, 69.2), turned to 90 degrees
- moved R2 72.1 mm to (118.1, 70.4)
- moved R7 71.6 mm to (113.3, 75.2)
- moved P8 70.7 mm to (165.0, 77.0), turned to 270 degrees
- moved R23 70.7 mm to (124.8, 77.5)
- moved R8 70.2 mm to (110.7, 77.0)
- moved R5 69.6 mm to (110.7, 78.4)
- moved R3 69.4 mm to (118.1, 72.0)
- moved P7 68.2 mm to (165.0, 88.0), turned to 270 degrees
- moved R21 67.0 mm to (112.6, 91.3)
- moved D8 66.2 mm to (120.8, 74.7), turned to 90 degrees
- moved R4 66.0 mm to (123.7, 71.6)
- moved R25 66.0 mm to (124.8, 78.9)
- moved R27 65.7 mm to (122.4, 77.5)
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
Commit message: Update circuitdiagram.
Parts:
- moved R22 30.0 mm to (116.6, 90.5), turned to 270 degrees
- moved SW2 27.1 mm to (149.4, 96.6)
- moved C9 21.4 mm to (125.7, 72.5), turned to 90 degrees
- moved R25 20.3 mm to (104.6, 78.1)
- moved U2 19.0 mm to (128.9, 72.5), turned to 270 degrees
- moved C5 17.4 mm to (123.6, 75.0), turned to 90 degrees
- moved C6 17.4 mm to (132.0, 72.5), turned to 90 degrees
- moved D6 17.4 mm to (112.5, 86.7), turned to 270 degrees
- moved R23 16.8 mm to (112.5, 88.9)
- moved R9 16.6 mm to (148.3, 72.4)
- moved P1 16.4 mm to (154.1, 73.3), turned to 270 degrees
- moved L1 15.5 mm to (148.1, 76.7), turned to 270 degrees
- moved C11 14.7 mm to (153.4, 79.6), turned to 180 degrees
- moved R17 14.4 mm to (139.6, 82.5)
- moved D4 14.1 mm to (136.7, 82.5), turned to 180 degrees
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Connections:
- D6 pad 1: Net-(D6-Pad1) -> /LED0
- D6 pad 2: /LED0 -> Net-(D6-Pad2)
- D7 pad 1: Net-(D7-Pad1) -> /LED1
- D7 pad 2: /LED1 -> Net-(D7-Pad2)
- D8 pad 1: Net-(D8-Pad1) -> /LED2
- D8 pad 2: /LED2 -> Net-(D8-Pad2)
- R23 pad 1: VCC -> GND
- R23 pad 2: Net-(D6-Pad1) -> Net-(D6-Pad2)
- R25 pad 1: VCC -> GND
- R25 pad 2: Net-(D7-Pad1) -> Net-(D7-Pad2)
- R27 pad 1: VCC -> GND
- R27 pad 2: Net-(D8-Pad1) -> Net-(D8-Pad2)
- U4 pad 13: /FR_ON -> /LS_ON
- U4 pad 22: /LS_ON -> /FR_ON
Routing:
- net GND: track 0.00 -> 294.3 mm, vias 0 -> 25
- net VCC: track 0.00 -> 108.9 mm, vias 0 -> 5
- net VEE: track 0.00 -> 103.3 mm, vias 0 -> 2
- net +BATT: track 0.00 -> 75.4 mm, vias 0 -> 4
- net /R_CW: track 0.00 -> 53.5 mm, vias 0 -> 4
- net /R_PULSE: track 0.00 -> 51.4 mm, vias 0 -> 4
- net /SLEEP: track 0.00 -> 50.2 mm, vias 0 -> 2
- net /L_CW: track 0.00 -> 45.3 mm, vias 0 -> 2
- net /PUSH_SW: track 0.00 -> 45.0 mm, vias 0 -> 2
- net /ENC_CLK: track 0.00 -> 43.8 mm, vias 0 -> 2
- net /L_PULSE: track 0.00 -> 43.2 mm, vias 0 -> 2
- net /ENC_MOSI: track 0.00 -> 40.6 mm, vias 0 -> 4
- net /LS_ON: track 0.00 -> 40.2 mm, vias 0 -> 2
- net /ENC_MISO: track 0.00 -> 38.1 mm, vias 0 -> 5
- net /FL_AD: track 0.00 -> 34.4 mm, vias 0 -> 3
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Other:
- net class Battery: clearance 0.254 -> 0.1524; trace_width 2 -> 0.5
- net class Bold: clearance 0.254 -> 0.1524; trace_width 1 -> 0.3
- net class Default: clearance 0.254 -> 0.1524
- rule trace_clearance: 0.254 -> 0.1524
- rule trace_min: 0.254 -> 0.1524

Commit message: fin
Routing:
- net GND: track 294.3 -> 319.5 mm, vias 25 -> 33
- net /R_PULSE: track 51.4 -> 54.9 mm
- net /LED2: track 20.7 -> 22.9 mm
- net /MD: track 14.2 -> 12.8 mm
- net /FR_AD: track 31.4 -> 30.1 mm, vias 3 -> 5
- net /RS_ON: track 31.7 -> 30.9 mm
- net /FR_ON: track 22.7 -> 22.0 mm
- added copper zone on B.Cu, net GND
- added copper zone on B.Cu, net Net-(P7-Pad6)
- added copper zone on B.Cu, net Net-(P8-Pad6)

Commit message: Order to elerow.
Routing:
- net GND: track 319.5 -> 323.1 mm
- net Net-(P8-Pad6): track 12.2 -> 15.4 mm
- net Net-(P7-Pad6): track 12.1 -> 15.3 mm
- net Net-(P8-Pad5): track 12.2 -> 14.9 mm
- net VCC: track 108.9 -> 111.1 mm
- net VEE: track 103.3 -> 103.8 mm
Changed lines of the file:
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@@
   (general
     (links 186)
-    (no_connects 8)
-    (area 99.949999 64.949999 167.680001 100.050001)
+    (no_connects 3)
+    (area 95.657999 62.383999 176.249001 102.335001)
     (thickness 1.6)
     (drawings 242)
-    (tracks 1244)
+    (tracks 1265)
     (zones 0)
     (modules 77)
@@
   (layers
     (0 F.Cu signal)
-    (31 B.Cu signal)
+    (31 B.Cu signal hide)
     (32 B.Adhes user)
     (33 F.Adhes user)
@@
     (visible_elements 7FFCF7FF)
     (pcbplotparams
-      (layerselection 0x00030_80000001)
+      (layerselection 0x010e0_80000001)
       (usegerberextensions true)
       (excludeedgelayer true)
@@
       (psa4output false)
       (plotreference true)
-      (plotvalue true)
+      (plotvalue false)
       (plotinvisibletext false)
       (padsonsilk false)
-      (subtractmaskfromsilk false)
+      (subtractmaskfromsilk true)
       (outputformat 1)
       (mirror false)
-      (drillshape 1)
+      (drillshape 0)
       (scaleselection 1)
-      (outputdirectory ""))
+      (outputdirectory product_data/))
   )
   (net 0 "")
@@
   (gr_line (start 136.779 82.4865) (end 176.149 82.4865) (angle 90) (layer Cmts.User) (width 0.2))
   (segment (start 137.7155 82.4865) (end 139.0865 82.4865) (width 0.254) (layer F.Cu) (net 1))
+  (segment (start 114.4016 95.8088) (end 114.4016 94.7674) (width 0.3) (layer F.Cu) (net 2))
+  (segment (start 114.4016 94.7674) (end 114.2326 94.9364) (width 0.3) (layer F.Cu) (net 2))
+  (segment (start 114.2326 94.9364) (end 113.03 94.9364) (width 0.3) (layer F.Cu) (net 2))
+  (segment (start 113.03 94.9364) (end 114.2326 94.9364) (width 0.3) (layer F.Cu) (net 2))
+  (segment (start 114.2326 94.9364) (end 114.4016 95.1054) (width 0.3) (layer F.Cu) (net 2))
+  (segment (start 114.4016 95.1054) (end 114.4016 95.8088) (width 0.3) (layer F.Cu) (net 2))
+  (segment (start 114.2326 94.9364) (end 114.4016 95.1054) (width 0.3) (layer F.Cu) (net 2))
+  (segment (start 114.4016 95.1054) (end 114.4016 95.8088) (width 0.3) (layer F.Cu) (net 2))
+  (segment (start 114.2326 94.9364) (end 114.4016 94.7674) (width 0.3) (layer F.Cu) (net 2))
   (segment (start 135.509 71.501) (end 137.541 71.501) (width 0.3) (layer F.Cu) (net 2))
   (segment (start 137.541 71.501) (end 137.5664 71.4756) (width 0.3) (layer F.Cu) (net 2))
@@
   (segment (start 121.666 93.8784) (end 118.4148 97.1296) (width 0.3) (layer B.Cu) (net 2))
   (via (at 114.4016 95.8088) (size 0.889) (drill 0.635) (layers F.Cu B.Cu) (net 2))
-  (segment (start 114.4016 95.8088) (end 114.4016 94.7674) (width 0.5) (layer F.Cu) (net 2))
-  (segment (start 113.03 94.9364) (end 114.2326 94.9364) (width 0.5) (layer F.Cu) (net 2))
   (segment (start 114.2326 94.9364) (end 114.4016 94.7674) (width 0.5) (layer F.Cu) (net 2))
   (segment (start 119.888 70.8025) (end 119.888 72.0725) (width 0.5) (layer F.Cu) (net 2))
@@
   (segment (start 133.096 80.3275) (end 133.096 78.486) (width 0.254) (layer B.Cu) (net 10))
   (segment (start 132.969 80.4545) (end 133.096 80.3275) (width 0.254) (layer B.Cu) (net 10))
+  (segment (start 137.7188 75.057) (end 137.7188 77.1812) (width 0.3) (layer F.Cu) (net 11))
+  (segment (start 137.7188 77.1812) (end 137.684 77.216) (width 0.3) (layer F.Cu) (net 11))
   (segment (start 117.9068 86.2076) (end 117.5004 86.2076) (width 0.3) (layer B.Cu) (net 11))
   (segment (start 121.6152 85.1408) (end 120.5484 86.2076) (width 0.3) (layer B.Cu) (net 11))
@@
   (segment (start 122.6145 85.1575) (end 122.6145 85.8012) (width 0.3) (layer F.Cu) (net 11))
   (segment (start 140.97 77.1525) (end 140.97 78.9305) (width 0.5) (layer F.Cu) (net 11))
-  (segment (start 137.684 75.057) (end 138.684 75.057) (width 0.5) (layer F.Cu) (net 11))
+  (segment (start 137.684 75.057) (end 137.7188 75.057) (width 0.5) (layer F.Cu) (net 11))
+  (segment (start 137.7188 75.057) (end 138.684 75.057) (width 0.5) (layer F.Cu) (net 11))
   (segment (start 140.081 74.549) (end 140.97 75.438) (width 0.5) (layer F.Cu) (net 11))
   (segment (start 139.192 74.549) (end 140.081 74.549) (width 0.5) (layer F.Cu) (net 11))
@@
   (segment (start 164.3028 88.986) (end 162.782 88.986) (width 0.254) (layer F.Cu) (net 17))
   (segment (start 164.7698 88.519) (end 164.3028 88.986) (width 0.254) (layer F.Cu) (net 17))
+  (segment (start 159.807 90.011) (end 159.807 87.925) (width 0.254) (layer F.Cu) (net 18))
+  (segment (start 159.568 87.686) (end 158.782 87.686) (width 0.254) (layer F.Cu) (net 18))
+  (segment (start 159.807 87.925) (end 159.568 87.686) (width 0.254) (layer F.Cu) (net 18))
   (segment (start 158.782 87.036) (end 158.782 85.1088) (width 0.254) (layer F.Cu) (net 18))
   (segment (start 164.5666 90.551) (end 164.5412 90.5256) (width 0.254) (layer F.Cu) (net 18))
@@
   (segment (start 164.0384 88.336) (end 162.782 88.336) (width 0.254) (layer F.Cu) (net 21))
   (segment (start 164.8714 87.503) (end 164.0384 88.336) (width 0.254) (layer F.Cu) (net 21))
+  (segment (start 158.782 77.287) (end 158.782 77.937) (width 0.254) (layer F.Cu) (net 22))
+  (segment (start 158.782 77.937) (end 158.782 79.9404) (width 0.254) (layer F.Cu) (net 22))
   (segment (start 160.457 78.962) (end 160.457 80.3656) (width 0.254) (layer F.Cu) (net 22))
   (segment (start 160.457 80.3656) (end 160.4264 80.3656) (width 0.254) (layer F.Cu) (net 22))
@@
   (segment (start 164.379 77.937) (end 162.782 77.937) (width 0.254) (layer F.Cu) (net 23))
   (segment (start 164.846 77.47) (end 164.379 77.937) (width 0.254) (layer F.Cu) (net 23))
+  (segment (start 159.807 78.962) (end 159.807 76.8506) (width 0.254) (layer F.Cu) (net 24))
+  (segment (start 159.5934 76.637) (end 158.782 76.637) (width 0.254) (layer F.Cu) (net 24))
+  (segment (start 159.807 76.8506) (end 159.5934 76.637) (width 0.254) (layer F.Cu) (net 24))
   (segment (start 158.782 75.987) (end 158.782 73.9836) (width 0.254) (layer F.Cu) (net 24))
   (via (at 164.4904 79.502) (size 0.889) (drill 0.635) (layers F.Cu B.Cu) (net 24))
@@
   (segment (start 125.73 69.4055) (end 123.994 71.1415) (width 0.254) (layer F.Cu) (net 28))
   (segment (start 123.994 71.1415) (end 123.994 71.501) (width 0.254) (layer F.Cu) (net 28))
+  (segment (start 110.236 90.8724) (end 110.236 91.1352) (width 0.3) (layer F.Cu) (net 29))
+  (segment (start 110.236 91.1352) (end 110.4392 91.3384) (width 0.3) (layer F.Cu) (net 29))
   (segment (start 115.5739 84.7305) (end 116.332 84.7305) (width 0.5) (layer F.Cu) (net 29))
   (segment (start 115.1636 85.1408) (end 115.5739 84.7305) (width 0.5) (layer F.Cu) (net 29))
@@
   (segment (start 109.0422 90.6526) (end 109.0168 90.6272) (width 0.5) (layer F.Cu) (net 29))
   (segment (start 111.1504 91.3384) (end 110.7948 91.3384) (width 0.5) (layer F.Cu) (net 29))
-  (segment (start 110.7948 91.3384) (end 109.728 91.3384) (width 0.5) (layer F.Cu) (net 29))
+  (segment (start 110.7948 91.3384) (end 110.4392 91.3384) (width 0.5) (layer F.Cu) (net 29))
+  (segment (start 110.4392 91.3384) (end 109.728 91.3384) (width 0.5) (layer F.Cu) (net 29))
   (segment (start 111.1504 91.3384) (end 115.1636 91.3384) (width 0.5) (layer F.Cu) (net 29))
   (segment (start 109.728 91.3384) (end 109.0168 90.6272) (width 0.5) (layer F.Cu) (net 29))
@@
   (segment (start 124.2988 93.8784) (end 124.5616 93.8784) (width 0.254) (layer F.Cu) (net 32))
   (segment (start 124.5616 93.8784) (end 126.238 95.5548) (width 0.254) (layer F.Cu) (net 32))
+  (segment (start 140.1865 82.4865) (end 140.8811 82.4865) (width 0.5) (layer F.Cu) (net 33))
+  (via (at 141.2875 80.5815) (size 0.889) (drill 0.635) (layers F.Cu B.Cu) (net 33))
+  (segment (start 142.0495 78.613) (end 143.0655 78.613) (width 0.5) (layer F.Cu) (net 33))
+  (via (at 142.0495 78.613) (size 0.889) (drill 0.635) (layers F.Cu B.Cu) (net 33))
+  (segment (start 141.2875 79.375) (end 142.0495 78.613) (width 0.5) (layer B.Cu) (net 33))
+  (segment (start 141.2875 80.5815) (end 141.2875 79.375) (width 0.5) (layer B.Cu) (net 33))
+  (segment (start 141.2875 82.0801) (end 141.2875 80.5815) (width 0.5) (layer F.Cu) (net 33))
+  (segment (start 140.8811 82.4865) (end 141.2875 82.0801) (width 0.5) (layer F.Cu) (net 33))
   (segment (start 122.47 74.4855) (end 122.47 73.5545) (width 0.5) (layer F.Cu) (net 33))
   (segment (start 122.6185 73.533) (end 122.555 73.4695) (width 0.5) (layer B.Cu) (net 33))
@@
   (segment (start 134.3025 73.533) (end 135.763 73.533) (width 0.5) (layer F.Cu) (net 33))
   (segment (start 134.2865 73.517) (end 134.3025 73.533) (width 0.5) (layer F.Cu) (net 33))
-  (segment (start 141.2875 80.5815) (end 141.2875 79.375) (width 0.5) (layer B.Cu) (net 33))
-  (segment (start 140.843 82.4865) (end 141.2875 82.042) (width 0.5) (layer F.Cu) (net 33))
-  (segment (start 141.2875 82.042) (end 141.2875 80.5815) (width 0.5) (layer F.Cu) (net 33))
-  (via (at 141.2875 80.5815) (size 0.889) (drill 0.635) (layers F.Cu B.Cu) (net 33))
-  (segment (start 140.1865 82.4865) (end 140.843 82.4865) (width 0.5) (layer F.Cu) (net 33))
-  (segment (start 142.0495 78.613) (end 143.0655 78.613) (width 0.5) (layer F.Cu) (net 33))
-  (via (at 142.0495 78.613) (size 0.889) (drill 0.635) (layers F.Cu B.Cu) (net 33))
-  (segment (start 141.2875 79.375) (end 142.0495 78.613) (width 0.5) (layer B.Cu) (net 33))
   (segment (start 143.0655 78.613) (end 142.875 78.613) (width 0.5) (layer F.Cu) (net 33))
   (segment (start 142.875 78.613) (end 143.0655 78.613) (width 0.5) (layer F.Cu) (net 33))
